File: Proyecto Final (PCB)/Proyecto Final.kicad_sch (KiCad schematic)
At the start: 61 parts, among them IC1 MC9S08MP16xLC, J1 Input, J10 Relay3, J11 Motor2, J12 Motor4, J13 LCD PINs, J14 Relay2, J15 Relay4, J16 PH_SENSOR, J17 Nivel_L, J18 Nivel_H, J19 Expansion2, J2 Luces_LEDs1, J20 Luces_LEDs2, J21 Conn_01x04_Male, J3 Expansions5, J4 DHT11_SENSOR, J5 LDR, J6 TDS_SENSOR, J7 Motor1, J8 Motor3, J9 Relay1, K1 FINDER-36.11, K2 FINDER-36.11, K3 FINDER-36.11, K4 FINDER-36.11, Q1 IRF3205, Q2 IRF3205, U1 AP63205WU, U2 MIC4427, U3 TLV2371D, U4 TLV2371D, U5 TLV2371D, U6 PC817, U7 PC817, U8 ULN2803A, Y1 Crystal

Commit message: 02/07/2022
Parts:
- removed U3, U4, U5: TLV2371D, Package_SO:SOIC-8_3.9x4.9mm_P1.27mm, symbol Amplifier_Operational:TLV2371D
- added C10, C11, C12: 100nF, Capacitor_SMD:C_0603_1608Metric, symbol Device:C
- added R15: 1k, Resistor_SMD:R_0603_1608Metric, symbol Device:R
- added R16, R17, R18, R19: 5k, Resistor_SMD:R_0603_1608Metric, symbol Device:R
- added RV1, RV2: 10k, Potentiometer_THT:Potentiometer_Bourns_3266Y_Vertical, symbol Device:R_Potentiometer
- added SW1: SWDIP, Button_Switch_THT:SW_DIP_SPSTx02_Slide_9.78x7.26mm_W7.62mm_P2.54mm, symbol Switch:SW_DIP_x02
- added U10: ULN2803A, Package_SO:SOIC-18W_7.5x11.6mm_P1.27mm, symbol Transistor_Array:ULN2803A
- added U3, U4: LM358, Package_SO:SOIC-8_3.9x4.9mm_P1.27mm, symbol Amplifier_Operational:LM358
- J21: footprint (none) -> Connector_PinHeader_1.00mm:PinHeader_1x04_P1.00mm_Vertical
- R10, R9: value 1k -> 5k
- Y1: footprint (none) -> Crystal:Crystal_HC49-4H_Vertical
Connections:
- net +12V: now also J2.2 (Pin_2), U10.10 (COM); no longer J2.1 (Pin_1)
- net +5V: now also C9.2, R10.1, R9.1, R16.1, R17.1, R18.1, R19.1, U3.8 (V+), U4.8 (V+)
- net ADC_e: now also C10.1, R15.1; no longer J3.5 (Pin_5)
- net GND: now also C9.1, C10.2, C11.1, C12.1, SW1.3, SW1.4, U10.9 (GND), U3.4 (V-), U4.4 (V-)
- net LEVEL_H: now also C12.2
- net LEVEL_L: now also C11.2
- net M1: now also U10.17 (O2), U10.18 (O1); no longer U8.14 (O5)
- net M2: now also U10.15 (O4), U10.16 (O3); no longer U8.13 (O6)
- net M3: now also U10.13 (O6), U10.14 (O5); no longer U8.12 (O7)
- net M4: now also U10.11 (O8), U10.12 (O7); no longer U8.11 (O8)
- net Motor1: now also IC1.23 (PTB4), U10.1 (I1), U10.2 (I2); no longer IC1.5 (PTC6), U8.4 (I4)
- net Motor2: now also IC1.16 (PTA7), U10.3 (I3), U10.4 (I4); no longer IC1.15 (PTA6), U8.3 (I3)
- net Motor3: now also IC1.15 (PTA6), U10.5 (I5), U10.6 (I6); no longer IC1.16 (PTA7), U8.2 (I2)
- net Motor4: now also IC1.5 (PTC6), U10.7 (I7), U10.8 (I8); no longer IC1.23 (PTB4), U8.1 (I1)
- net Relay1: now also U8.4 (I4); no longer U8.8 (I8)
- net Relay2: now also U8.3 (I3); no longer U8.7 (I7)
- net Relay3: now also U8.2 (I2); no longer U8.6 (I6)
- net Relay4: now also U8.1 (I1); no longer U8.5 (I5)
- net Rx: now also R18.2
- net SCL: now also J3.3 (Pin_3), R17.2
- net SDA: now also J3.4 (Pin_4), R16.2
- net Tx: now also R19.2
- net at R4.2: now also U3.1, U3.2 (-)
- net at J18.2 (Pin_2): now also RV2.3; no longer R10.2
- net at U7.1: now also RV2.1, RV2.2; no longer R10.1
- net at J16.3 (Pin_3): now also U4.3 (+)
- net at U6.1: now also RV1.1, RV1.2; no longer R9.1
- net at R6.2: now also U4.1, U4.2 (-)
- net at J17.2 (Pin_2): now also RV1.3; no longer R9.2
- net at J6.3 (Pin_3): now also U4.5 (+)
- net at Q1.2 (D): now also J2.1 (Pin_1); no longer J2.2 (Pin_2)
- net at R5.2: now also U4.6 (-), U4.7
- net at J5.2 (Pin_2): now also U3.3 (+)
- net PTC0 renamed PWM_L2
- net PTC1 renamed PWM_L1
- net SCL_e renamed DIP2
- net DIP2: now also R9.2, SW1.2; no longer J3.4 (Pin_4)
- net SDA_e renamed DIP1
- net DIP1: now also R10.2, SW1.1; no longer J3.3 (Pin_3)
- new net: J3.5 (Pin_5), U3.5 (+)
- new net: R15.2, U3.6 (-), U3.7
- no-connect marks 0 -> 8
Other:
- note added: "DSW"
- note removed: "Pull-up"
- moved on the sheet: J17, J18, J19, J2, J3, R7, R8, U6, U7, U8

Commit message: 08/07/2022
Parts:
- added C? (x2): 30pF, Capacitor_SMD:C_0603_1608Metric, symbol Device:C
- added U?: ULN2003A, symbol Transistor_Array:ULN2003A
- L1: footprint Inductor_SMD:L_0603_1608Metric -> Inductor_SMD:L_Bourns_SRN6045TA
Connections:
- net GND: now also C?.1, C?.1
- net at IC1.27 (PTE5/XTAL), Y1.2: now also C?.2
- net at IC1.28 (PTE6/EXTAL), Y1.1: now also C?.2
- no-connect marks 8 -> 24
Changed lines of the file:
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@@
   (junction (at 220.98 110.49) (diameter 0) (color 0 0 0 0)
   )
+  (junction (at 177.8 166.37) (diameter 0) (color 0 0 0 0)
+  )
+  (junction (at 177.8 156.21) (diameter 0) (color 0 0 0 0)
+  )
   (junction (at 361.95 60.96) (diameter 0) (color 0 0 0 0)
   )
@@
   (no_connect (at 388.62 191.77))
   (no_connect (at 388.62 189.23))
+  (no_connect (at 344.17 176.53))
+  (no_connect (at 344.17 181.61))
+  (no_connect (at 344.17 184.15))
+  (no_connect (at 344.17 186.69))
+  (no_connect (at 344.17 189.23))
+  (no_connect (at 344.17 191.77))
+  (no_connect (at 344.17 194.31))
+  (no_connect (at 344.17 196.85))
+  (no_connect (at 334.01 201.93))
+  (no_connect (at 323.85 194.31))
+  (no_connect (at 323.85 196.85))
+  (no_connect (at 323.85 181.61))
+  (no_connect (at 323.85 184.15))
+  (no_connect (at 323.85 186.69))
+  (no_connect (at 323.85 189.23))
+  (no_connect (at 323.85 191.77))
   (wire (pts (xy 115.57 38.1) (xy 115.57 31.75))
     (stroke (width 0) (type default) (color 0 0 0 0))
@@
     (stroke (width 0) (type default) (color 0 0 0 0))
   )
+  (wire (pts (xy 162.56 157.48) (xy 162.56 156.21))
+    (stroke (width 0) (type default) (color 0 0 0 0))
+  )
   (wire (pts (xy 354.33 146.05) (xy 354.33 147.32))
     (stroke (width 0) (type default) (color 0 0 0 0))
@@
     (stroke (width 0) (type default) (color 0 0 0 0))
   )
+  (wire (pts (xy 162.56 167.64) (xy 162.56 166.37))
+    (stroke (width 0) (type default) (color 0 0 0 0))
+  )
   (wire (pts (xy 394.97 231.14) (xy 391.16 231.14))
     (stroke (width 0) (type default) (color 0 0 0 0))
@@
     (stroke (width 0) (type default) (color 0 0 0 0))
   )
+  (wire (pts (xy 172.72 156.21) (xy 177.8 156.21))
+    (stroke (width 0) (type default) (color 0 0 0 0))
+  )
   (wire (pts (xy 57.15 248.92) (xy 57.15 259.08))
     (stroke (width 0) (type default) (color 0 0 0 0))
@@
     (stroke (width 0) (type default) (color 0 0 0 0))
   )
+  (wire (pts (xy 162.56 166.37) (xy 165.1 166.37))
+    (stroke (width 0) (type default) (color 0 0 0 0))
+  )
+  (wire (pts (xy 162.56 156.21) (xy 165.1 156.21))
+    (stroke (width 0) (type default) (color 0 0 0 0))
+  )
   (wire (pts (xy 229.87 248.92) (xy 229.87 251.46))
     (stroke (width 0) (type default) (color 0 0 0 0))
@@
     (stroke (width 0) (type default) (color 0 0 0 0))
   )
+  (wire (pts (xy 172.72 166.37) (xy 177.8 166.37))
+    (stroke (width 0) (type default) (color 0 0 0 0))
+  )
   (wire (pts (xy 207.01 29.21) (xy 208.28 29.21))
     (stroke (width 0) (type default) (color 0 0 0 0))
@@
     (pin "8")
   )
+  (symbol (lib_id "Transistor_Array:ULN2003A") (at 334.01 186.69 0) (unit 1)
+    (in_bom yes) (on_board yes) (fields_autoplaced)
+    (property "Reference" "U?" (id 0) (at 334.01 168.91 0))
+    (property "Value" "ULN2003A" (id 1) (at 334.01 171.45 0))
+    (property "Footprint" "" (id 2) (at 335.28 200.66 0)
+      (effects (font (size 1.27 1.27)) (justify left) hide)
+    )
+    (property "Datasheet" "http://www.ti.com/lit/ds/symlink/uln2003a.pdf" (id 3) (at 336.55 191.77 0)
+      (effects (font (size 1.27 1.27)) hide)
+    )
+    (pin "1")
+    (pin "10")
+    (pin "11")
+    (pin "12")
+    (pin "13")
+    (pin "14")
+    (pin "15")
+    (pin "16")
+    (pin "2")
+    (pin "3")
+    (pin "4")
+    (pin "5")
+    (pin "6")
+    (pin "7")
+    (pin "8")
+    (pin "9")
+  )
   (symbol (lib_id "power:GND") (at 173.99 38.1 0) (unit 1)
     (in_bom yes) (on_board yes)
@@
     (property "Reference" "L1" (id 0) (at 76.2 19.05 90))
     (property "Value" "4.7uH" (id 1) (at 76.2 21.59 90))
-    (property "Footprint" "Inductor_SMD:L_0603_1608Metric" (id 2) (at 76.2 25.4 0)
+    (property "Footprint" "Inductor_SMD:L_Bourns_SRN6045TA" (id 2) (at 76.2 25.4 0)
       (effects (font (size 1.27 1.27)) hide)
     )
@@
     (pin "2")
   )
+  (symbol (lib_id "Device:C") (at 168.91 156.21 90) (unit 1)
+    (in_bom yes) (on_board yes)
+    (property "Reference" "C?" (id 0) (at 170.18 149.86 0)
+      (effects (font (size 1.27 1.27)) (justify right))
+    )
+    (property "Value" "30pF" (id 1) (at 167.64 147.32 0)
+      (effects (font (size 1.27 1.27)) (justify right))
+    )
+    (property "Footprint" "Capacitor_SMD:C_0603_1608Metric" (id 2) (at 172.72 155.2448 0)
+      (effects (font (size 1.27 1.27)) hide)
+    )
+    (property "Datasheet" "~" (id 3) (at 168.91 156.21 0)
+      (effects (font (size 1.27 1.27)) hide)
+    )
+    (pin "1")
+    (pin "2")
+  )
   (symbol (lib_id "Device:C") (at 36.83 35.56 0) (unit 1)
     (in_bom yes) (on_board yes) (fields_autoplaced)
@@
     (pin "1")
   )
+  (symbol (lib_id "power:GND") (at 162.56 167.64 0) (unit 1)
+    (in_bom yes) (on_board yes)
+    (property "Reference" "#PWR?" (id 0) (at 162.56 173.99 0)
+      (effects (font (size 1.27 1.27)) hide)
+    )
+    (property "Value" "GND" (id 1) (at 162.56 171.45 0))
+    (property "Footprint" "" (id 2) (at 162.56 167.64 0)
+      (effects (font (size 1.27 1.27)) hide)
+    )
+    (property "Datasheet" "" (id 3) (at 162.56 167.64 0)
+      (effects (font (size 1.27 1.27)) hide)
+    )
+    (pin "1")
+  )
   (symbol (lib_id "Device:C") (at 88.9 34.29 0) (unit 1)
     (in_bom yes) (on_board yes)
@@
     (pin "2")
   )
+  (symbol (lib_id "Device:C") (at 168.91 166.37 90) (unit 1)
+    (in_bom yes) (on_board yes)
+    (property "Reference" "C?" (id 0) (at 170.18 170.18 0)
+      (effects (font (size 1.27 1.27)) (justify right))
+    )
+    (property "Value" "30pF" (id 1) (at 167.64 170.18 0)
+      (effects (font (size 1.27 1.27)) (justify right))
+    )
+    (property "Footprint" "Capacitor_SMD:C_0603_1608Metric" (id 2) (at 172.72 165.4048 0)
+      (effects (font (size 1.27 1.27)) hide)
+    )
+    (property "Datasheet" "~" (id 3) (at 168.91 166.37 0)
+      (effects (font (size 1.27 1.27)) hide)
+    )
+    (pin "1")
+    (pin "2")
+  )
   (symbol (lib_id "Device:R") (at 285.75 29.21 90) (unit 1)
     (in_bom yes) (on_board yes) (fields_autoplaced)
@@
     (pin "A2")
   )
+  (symbol (lib_id "power:GND") (at 162.56 157.48 0) (unit 1)
+    (in_bom yes) (on_board yes)
+    (property "Reference" "#PWR?" (id 0) (at 162.56 163.83 0)
+      (effects (font (size 1.27 1.27)) hide)
+    )
+    (property "Value" "GND" (id 1) (at 162.56 161.29 0))
+    (property "Footprint" "" (id 2) (at 162.56 157.48 0)
+      (effects (font (size 1.27 1.27)) hide)
+    )
+    (property "Datasheet" "" (id 3) (at 162.56 157.48 0)
+      (effects (font (size 1.27 1.27)) hide)
+    )
+    (pin "1")
+  )
   (symbol (lib_id "power:+5V") (at 359.41 77.47 90) (unit 1)
     (in_bom yes) (on_board yes)
@@
       (reference "#PWR0143") (unit 1) (value "+12V") (footprint "")
     )
+    (path "/77c996a0-124a-4123-b417-fc3db2d2b43c"
+      (reference "#PWR?") (unit 1) (value "GND") (footprint "")
+    )
+    (path "/d71249f4-58a6-4fe5-88d7-9ef835ef09a3"
+      (reference "#PWR?") (unit 1) (value "GND") (footprint "")
+    )
     (path "/426351f6-319f-45ba-aa2a-dad65db32d2c"
       (reference "C1") (unit 1) (value "10uF") (footprint "Capacitor_SMD:C_0603_1608Metric")
@@
       (reference "C12") (unit 1) (value "100nF") (footprint "Capacitor_SMD:C_0603_1608Metric")
     )
+    (path "/424fc4d7-c4ad-45ef-9ea9-15160714ce70"
+      (reference "C?") (unit 1) (value "30pF") (footprint "Capacitor_SMD:C_0603_1608Metric")
+    )
+    (path "/995b9dc9-6dc1-4f0e-9472-f909ef2b6010"
+      (reference "C?") (unit 1) (value "30pF") (footprint "Capacitor_SMD:C_0603_1608Metric")
+    )
     (path "/48ba80f7-2e65-4f1a-8f71-21ac0eb2c29d"
       (reference "IC1") (unit 1) (value "MC9S08MP16xLC") (footprint "Package_QFP:LQFP-32_7x7mm_P0.8mm")
@@
     )
     (path "/31acafcc-16ba-4e90-8ba9-241fa4166c21"
-      (reference "L1") (unit 1) (value "4.7uH") (footprint "Inductor_SMD:L_0603_1608Metric")
+      (reference "L1") (unit 1) (value "4.7uH") (footprint "Inductor_SMD:L_Bourns_SRN6045TA")
     )
     (path "/952c7ee3-e506-4659-ab8b-44adb1c42123"
@@
       (reference "U10") (unit 1) (value "ULN2803A") (footprint "Package_SO:SOIC-18W_7.5x11.6mm_P1.27mm")
     )
+    (path "/062d7b44-e29e-4d8b-b3eb-fb01cbd8354b"
+      (reference "U?") (unit 1) (value "ULN2003A") (footprint "")
+    )
     (path "/e550df42-ddf7-4405-a18f-e433860943e4"

Commit message: 08/07/2022
Parts:
- J13, J21: footprint Connector_PinHeader_1.00mm:PinHeader_1x04_P1.00mm_Vertical -> Connector_PinHeader_2.54mm:PinHeader_1x04_P2.54mm_Vertical
- gave numbers to parts that had none: 3
Changed lines of the file:
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@@
   (symbol (lib_id "Transistor_Array:ULN2003A") (at 334.01 186.69 0) (unit 1)
     (in_bom yes) (on_board yes) (fields_autoplaced)
-    (property "Reference" "U?" (id 0) (at 334.01 168.91 0))
+    (property "Reference" "U5" (id 0) (at 334.01 168.91 0))
     (property "Value" "ULN2003A" (id 1) (at 334.01 171.45 0))
     (property "Footprint" "" (id 2) (at 335.28 200.66 0)
@@
     (property "Reference" "J21" (id 0) (at 184.785 139.7 0))
     (property "Value" "Conn_01x04_Male" (id 1) (at 184.785 142.24 0))
-    (property "Footprint" "Connector_PinHeader_1.00mm:PinHeader_1x04_P1.00mm_Vertical" (id 2) (at 184.15 147.32 0)
+    (property "Footprint" "Connector_PinHeader_2.54mm:PinHeader_1x04_P2.54mm_Vertical" (id 2) (at 184.15 147.32 0)
       (effects (font (size 1.27 1.27)) hide)
     )
@@
   (symbol (lib_id "Device:C") (at 168.91 156.21 90) (unit 1)
     (in_bom yes) (on_board yes)
-    (property "Reference" "C?" (id 0) (at 170.18 149.86 0)
+    (property "Reference" "C13" (id 0) (at 170.18 149.86 0)
       (effects (font (size 1.27 1.27)) (justify right))
     )
@@
   (symbol (lib_id "power:GND") (at 162.56 167.64 0) (unit 1)
     (in_bom yes) (on_board yes)
-    (property "Reference" "#PWR?" (id 0) (at 162.56 173.99 0)
+    (property "Reference" "#PWR0112" (id 0) (at 162.56 173.99 0)
       (effects (font (size 1.27 1.27)) hide)
     )
@@
   (symbol (lib_id "Device:C") (at 168.91 166.37 90) (unit 1)
     (in_bom yes) (on_board yes)
-    (property "Reference" "C?" (id 0) (at 170.18 170.18 0)
+    (property "Reference" "C14" (id 0) (at 170.18 170.18 0)
       (effects (font (size 1.27 1.27)) (justify right))
     )
@@
     (property "Reference" "J13" (id 0) (at 391.16 146.05 0))
     (property "Value" "LCD PINs" (id 1) (at 392.43 148.59 0))
-    (property "Footprint" "Connector_PinHeader_1.00mm:PinHeader_1x04_P1.00mm_Vertical" (id 2) (at 388.62 153.67 0)
+    (property "Footprint" "Connector_PinHeader_2.54mm:PinHeader_1x04_P2.54mm_Vertical" (id 2) (at 388.62 153.67 0)
       (effects (font (size 1.27 1.27)) hide)
     )
@@
   (symbol (lib_id "power:GND") (at 162.56 157.48 0) (unit 1)
     (in_bom yes) (on_board yes)
-    (property "Reference" "#PWR?" (id 0) (at 162.56 163.83 0)
+    (property "Reference" "#PWR0113" (id 0) (at 162.56 163.83 0)
       (effects (font (size 1.27 1.27)) hide)
     )
@@
       (reference "#PWR0111") (unit 1) (value "+5V") (footprint "")
     )
+    (path "/77c996a0-124a-4123-b417-fc3db2d2b43c"
+      (reference "#PWR0112") (unit 1) (value "GND") (footprint "")
+    )
+    (path "/d71249f4-58a6-4fe5-88d7-9ef835ef09a3"
+      (reference "#PWR0113") (unit 1) (value "GND") (footprint "")
+    )
     (path "/46e82a5d-9f45-4a44-994e-24fb5f2b374a"
       (reference "#PWR0114") (unit 1) (value "GND") (footprint "")
@@
       (reference "#PWR0143") (unit 1) (value "+12V") (footprint "")
     )
-    (path "/77c996a0-124a-4123-b417-fc3db2d2b43c"
-      (reference "#PWR?") (unit 1) (value "GND") (footprint "")
-    )
-    (path "/d71249f4-58a6-4fe5-88d7-9ef835ef09a3"
-      (reference "#PWR?") (unit 1) (value "GND") (footprint "")
-    )
     (path "/426351f6-319f-45ba-aa2a-dad65db32d2c"
       (reference "C1") (unit 1) (value "10uF") (footprint "Capacitor_SMD:C_0603_1608Metric")
@@
     )
     (path "/424fc4d7-c4ad-45ef-9ea9-15160714ce70"
-      (reference "C?") (unit 1) (value "30pF") (footprint "Capacitor_SMD:C_0603_1608Metric")
+      (reference "C13") (unit 1) (value "30pF") (footprint "Capacitor_SMD:C_0603_1608Metric")
     )
     (path "/995b9dc9-6dc1-4f0e-9472-f909ef2b6010"
-      (reference "C?") (unit 1) (value "30pF") (footprint "Capacitor_SMD:C_0603_1608Metric")
+      (reference "C14") (unit 1) (value "30pF") (footprint "Capacitor_SMD:C_0603_1608Metric")
     )
     (path "/48ba80f7-2e65-4f1a-8f71-21ac0eb2c29d"
@@
     )
     (path "/b9a0f191-d2e7-4c7c-b85b-a2280cdf7a93"
-      (reference "J13") (unit 1) (value "LCD PINs") (footprint "Connector_PinHeader_1.00mm:PinHeader_1x04_P1.00mm_Vertical")
+      (reference "J13") (unit 1) (value "LCD PINs") (footprint "Connector_PinHeader_2.54mm:PinHeader_1x04_P2.54mm_Vertical")
     )
     (path "/8125caf4-34cd-4456-8a7e-9eba6d909ba0"
@@
     )
     (path "/0d05dfe4-0904-428f-9297-a9375e9effd8"
-      (reference "J21") (unit 1) (value "Conn_01x04_Male") (footprint "Connector_PinHeader_1.00mm:PinHeader_1x04_P1.00mm_Vertical")
+      (reference "J21") (unit 1) (value "Conn_01x04_Male") (footprint "Connector_PinHeader_2.54mm:PinHeader_1x04_P2.54mm_Vertical")
     )
     (path "/d5b17a47-b3c9-42ee-b747-5fa759911505"
@@
       (reference "U4") (unit 3) (value "LM358") (footprint "")
     )
+    (path "/062d7b44-e29e-4d8b-b3eb-fb01cbd8354b"
+      (reference "U5") (unit 1) (value "ULN2003A") (footprint "")
+    )
     (path "/2bb410d4-2f63-4326-b5d1-6e6cc4103f9a"
       (reference "U6") (unit 1) (value "PC817") (footprint "Package_DIP:DIP-4_W7.62mm")
@@
       (reference "U10") (unit 1) (value "ULN2803A") (footprint "Package_SO:SOIC-18W_7.5x11.6mm_P1.27mm")
     )
-    (path "/062d7b44-e29e-4d8b-b3eb-fb01cbd8354b"
-      (reference "U?") (unit 1) (value "ULN2003A") (footprint "")
-    )
     (path "/e550df42-ddf7-4405-a18f-e433860943e4"

Commit message: 14/07/2022
Parts:
- removed C1: 10uF, Capacitor_SMD:C_0603_1608Metric, symbol Device:C
- removed C10, C11, C12, C2, C5, C7, C8: 100nF, Capacitor_SMD:C_0603_1608Metric, symbol Device:C
- removed C3: 22uF, Capacitor_SMD:C_0603_1608Metric, symbol Device:C
- removed C4: 22uf, Capacitor_SMD:C_0603_1608Metric, symbol Device:C
- removed J10: Relay3, TerminalBlock:TerminalBlock_bornier-3_P5.08mm, symbol Connector_Generic:Conn_01x03
- removed J11: Motor2, TerminalBlock:TerminalBlock_bornier-2_P5.08mm, symbol Connector_Generic:Conn_01x02
- removed J12: Motor4, TerminalBlock:TerminalBlock_bornier-2_P5.08mm, symbol Connector_Generic:Conn_01x02
- removed J13: LCD PINs, Connector_PinHeader_2.54mm:PinHeader_1x04_P2.54mm_Vertical, symbol Connector:Conn_01x04_Male
- removed J14: Relay2, TerminalBlock:TerminalBlock_bornier-3_P5.08mm, symbol Connector_Generic:Conn_01x03
- removed J15: Relay4, TerminalBlock:TerminalBlock_bornier-3_P5.08mm, symbol Connector_Generic:Conn_01x03
- removed J16: PH_SENSOR, TerminalBlock:TerminalBlock_bornier-3_P5.08mm, symbol Connector_Generic:Conn_01x03
- removed J17: Nivel_L, TerminalBlock:TerminalBlock_bornier-2_P5.08mm, symbol Connector_Generic:Conn_01x02
- removed J18: Nivel_H, TerminalBlock:TerminalBlock_bornier-2_P5.08mm, symbol Connector_Generic:Conn_01x02
- removed J19: Expansion2, TerminalBlock:TerminalBlock_bornier-2_P5.08mm, symbol Connector_Generic:Conn_01x02
- removed J2: Luces_LEDs1, TerminalBlock:TerminalBlock_bornier-2_P5.08mm, symbol Connector_Generic:Conn_01x02
- removed J20: Luces_LEDs2, TerminalBlock:TerminalBlock_bornier-2_P5.08mm, symbol Connector_Generic:Conn_01x02
- removed J3: Expansions5, TerminalBlock:TerminalBlock_bornier-5_P5.08mm, symbol Connector_Generic:Conn_01x05
- removed J4: DHT11_SENSOR, TerminalBlock:TerminalBlock_bornier-3_P5.08mm, symbol Connector_Generic:Conn_01x03
- removed J5: LDR, TerminalBlock:TerminalBlock_bornier-2_P5.08mm, symbol Connector_Generic:Conn_01x02
- removed J6: TDS_SENSOR, TerminalBlock:TerminalBlock_bornier-3_P5.08mm, symbol Connector_Generic:Conn_01x03
- removed J7: Motor1, TerminalBlock:TerminalBlock_bornier-2_P5.08mm, symbol Connector_Generic:Conn_01x02
- removed J8: Motor3, TerminalBlock:TerminalBlock_bornier-2_P5.08mm, symbol Connector_Generic:Conn_01x02
- removed J9: Relay1, TerminalBlock:TerminalBlock_bornier-3_P5.08mm, symbol Connector_Generic:Conn_01x03
- removed K1, K2, K3, K4: FINDER-36.11, Relay_THT:Relay_SPDT_Finder_36.11, symbol Relay:FINDER-36.11
- removed L1: 4.7uH, Inductor_SMD:L_Bourns_SRN6045TA, symbol Device:L
- removed Q1, Q2: IRF3205, Package_TO_SOT_THT:TO-220-3_Vertical, symbol Transistor_FET:IRF3205
- removed R1, R13, R14, R2: 10, Resistor_SMD:R_0603_1608Metric, symbol Device:R
- removed R11, R12: 10k, Resistor_SMD:R_0603_1608Metric, symbol Device:R
- removed R15, R4, R5, R6: 1k, Resistor_SMD:R_0603_1608Metric, symbol Device:R
- removed R16, R17, R18, R19, R3, R7, R8: 5k, Resistor_SMD:R_0603_1608Metric, symbol Device:R
- removed RV1, RV2: 10k, Potentiometer_THT:Potentiometer_Bourns_3266Y_Vertical, symbol Device:R_Potentiometer
- removed U1: AP63205WU, Package_TO_SOT_SMD:TSOT-23-6, symbol Regulator_Switching:AP63205WU
- removed U10, U8: ULN2803A, Package_SO:SOIC-18W_7.5x11.6mm_P1.27mm, symbol Transistor_Array:ULN2803A
- removed U2: MIC4427, Package_SO:SOIC-8_3.9x4.9mm_P1.27mm, symbol Driver_FET:MIC4427
- removed U3, U4: LM358, Package_SO:SOIC-8_3.9x4.9mm_P1.27mm, symbol Amplifier_Operational:LM358
- removed U5: ULN2003A, symbol Transistor_Array:ULN2003A
- removed U6, U7: PC817, Package_DIP:DIP-4_W7.62mm, symbol Isolator:PC817
- added R20: 1M, Resistor_SMD:R_0201_0603Metric, symbol Device:R
Connections:
- net at C13.2, IC1.27 (PTE5/XTAL), Y1.2: now also R20.2
- net at C14.2, IC1.28 (PTE6/EXTAL), Y1.1: now also R20.1
- no-connect marks 24 -> 0
Other:
- added sheet Expansions (Expansion_Header.kicad_sch)
- added sheet Fuente SW (Regulador 5V 2A.kicad_sch)
- added sheet Lcd (LCD Header.kicad_sch)
- added sheet MOSFET Driver (MIC 4427.kicad_sch)
- added sheet Motor Driver (ULN2003A.kicad_sch)
- added sheet Relay Modules (ULN.kicad_sch)
- added sheet Sensors (Comp & LPF.kicad_sch)
- note added: "Expansiones"
- note added: "LCD Header"
- note added: "Motor Driver"
- note added: "Sensons Input"
- note added: "Voltage Input"
- note removed: "Driver"
- note removed: "Expansions"
- note removed: "Input"
- note removed: "LCD"
- note removed: "Motors"
- note removed: "Relay Outputs"
- note removed: "Sensors"
- moved on the sheet: C13, C14, C6, C9, IC1, J1, J21, R10, R9, SW1, Y1
