File: Proyecto Final (PCB)/Proyecto Final.kicad_sch (KiCad schematic)
At the start: 12 parts, among them IC1 MC9S08MP16xLC, J1 Input, J21 Conn_01x04_Male, SW1 SWDIP, Y1 Crystal

Commit message: 15/07/2022
Parts:
- added L2: 27n, Inductor_SMD:L_0805_2012Metric, symbol Device:L
- added RV3: Varistor_6V, Capacitor_SMD:C_0805_2012Metric, symbol Device:Varistor
Connections:
- net +5V: now also L2.2, RV3.1; no longer C9.2, IC1.21 (VDDA/VREFH)
- net GND: now also RV3.2
- new net: C9.2, IC1.21 (VDDA/VREFH), L2.1
Changed lines of the file:
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@@
   (junction (at 172.72 124.46) (diameter 0) (color 0 0 0 0)
   )
+  (junction (at 69.85 68.58) (diameter 0) (color 0 0 0 0)
+  )
+  (junction (at 190.5 68.58) (diameter 0) (color 0 0 0 0)
+  )
+  (junction (at 62.23 71.12) (diameter 0) (color 0 0 0 0)
+  )
+  (junction (at 88.9 71.12) (diameter 0) (color 0 0 0 0)
+  )
   (junction (at 214.63 68.58) (diameter 0) (color 0 0 0 0)
   )
-  (junction (at 69.85 68.58) (diameter 0) (color 0 0 0 0)
-  )
-  (junction (at 62.23 71.12) (diameter 0) (color 0 0 0 0)
-  )
-  (junction (at 88.9 71.12) (diameter 0) (color 0 0 0 0)
-  )
   (junction (at 172.72 114.3) (diameter 0) (color 0 0 0 0)
   )
@@
     (stroke (width 0) (type default) (color 0 0 0 0))
   )
+  (wire (pts (xy 214.63 64.77) (xy 214.63 68.58))
+    (stroke (width 0) (type default) (color 0 0 0 0))
+  )
   (polyline (pts (xy 92.71 151.13) (xy 129.54 151.13))
     (stroke (width 0) (type default) (color 0 0 0 0))
@@
     (stroke (width 0) (type default) (color 0 0 0 0))
   )
-  (wire (pts (xy 200.66 68.58) (xy 204.47 68.58))
+  (wire (pts (xy 182.88 68.58) (xy 190.5 68.58))
     (stroke (width 0) (type default) (color 0 0 0 0))
   )
@@
     (stroke (width 0) (type default) (color 0 0 0 0))
   )
+  (wire (pts (xy 190.5 64.77) (xy 190.5 68.58))
+    (stroke (width 0) (type default) (color 0 0 0 0))
+  )
   (polyline (pts (xy 91.44 115.57) (xy 91.44 81.28))
     (stroke (width 0) (type default) (color 0 0 0 0))
@@
     (stroke (width 0) (type default) (color 0 0 0 0))
   )
+  (wire (pts (xy 231.14 68.58) (xy 233.68 68.58))
+    (stroke (width 0) (type default) (color 0 0 0 0))
+  )
   (polyline (pts (xy 92.71 45.72) (xy 129.54 45.72))
     (stroke (width 0) (type default) (color 0 0 0 0))
@@
     (stroke (width 0) (type default) (color 0 0 0 0))
   )
+  (wire (pts (xy 214.63 68.58) (xy 223.52 68.58))
+    (stroke (width 0) (type default) (color 0 0 0 0))
+  )
   (wire (pts (xy 237.49 118.11) (xy 250.19 118.11))
     (stroke (width 0) (type default) (color 0 0 0 0))
@@
     (stroke (width 0) (type default) (color 0 0 0 0))
   )
+  (wire (pts (xy 190.5 68.58) (xy 204.47 68.58))
+    (stroke (width 0) (type default) (color 0 0 0 0))
+  )
+  (wire (pts (xy 190.5 54.61) (xy 190.5 57.15))
+    (stroke (width 0) (type default) (color 0 0 0 0))
+  )
   (polyline (pts (xy 52.07 115.57) (xy 52.07 81.28))
     (stroke (width 0) (type default) (color 0 0 0 0))
@@
     (stroke (width 0) (type default) (color 0 0 0 0))
   )
-  (wire (pts (xy 214.63 69.85) (xy 214.63 68.58))
-    (stroke (width 0) (type default) (color 0 0 0 0))
-  )
   (wire (pts (xy 161.29 124.46) (xy 161.29 123.19))
     (stroke (width 0) (type default) (color 0 0 0 0))
@@
     (stroke (width 0) (type default) (color 0 0 0 0))
   )
-  (wire (pts (xy 214.63 64.77) (xy 214.63 68.58))
-    (stroke (width 0) (type default) (color 0 0 0 0))
-  )
   (wire (pts (xy 172.72 90.17) (xy 181.61 90.17))
     (stroke (width 0) (type default) (color 0 0 0 0))
@@
     (stroke (width 0) (type default) (color 0 0 0 0))
   )
+  (wire (pts (xy 214.63 68.58) (xy 214.63 69.85))
+    (stroke (width 0) (type default) (color 0 0 0 0))
+  )
   (wire (pts (xy 172.72 82.55) (xy 181.61 82.55))
-    (stroke (width 0) (type default) (color 0 0 0 0))
-  )
-  (wire (pts (xy 214.63 68.58) (xy 204.47 68.58))
     (stroke (width 0) (type default) (color 0 0 0 0))
   )
@@
     )
     (pin "1")
+  )
+  (symbol (lib_id "Device:L") (at 227.33 68.58 90) (unit 1)
+    (in_bom yes) (on_board yes) (fields_autoplaced)
+    (property "Reference" "L2" (id 0) (at 227.33 62.23 90))
+    (property "Value" "27n" (id 1) (at 227.33 64.77 90))
+    (property "Footprint" "Inductor_SMD:L_0805_2012Metric" (id 2) (at 227.33 68.58 0)
+      (effects (font (size 1.27 1.27)) hide)
+    )
+    (property "Datasheet" "~" (id 3) (at 227.33 68.58 0)
+      (effects (font (size 1.27 1.27)) hide)
+    )
+    (pin "1")
+    (pin "2")
   )
   (symbol (lib_id "power:GND") (at 204.47 54.61 180) (unit 1)
@@
     (pin "2")
   )
-  (symbol (lib_id "power:+5V") (at 200.66 68.58 90) (mirror x) (unit 1)
-    (in_bom yes) (on_board yes)
-    (property "Reference" "#PWR03" (id 0) (at 204.47 68.58 0)
-      (effects (font (size 1.27 1.27)) hide)
-    )
-    (property "Value" "+5V" (id 1) (at 196.85 68.58 0))
-    (property "Footprint" "" (id 2) (at 200.66 68.58 0)
-      (effects (font (size 1.27 1.27)) hide)
-    )
-    (property "Datasheet" "" (id 3) (at 200.66 68.58 0)
+  (symbol (lib_id "Device:Varistor") (at 190.5 60.96 0) (mirror x) (unit 1)
+    (in_bom yes) (on_board yes) (fields_autoplaced)
+    (property "Reference" "RV3" (id 0) (at 186.69 59.4367 0)
+      (effects (font (size 1.27 1.27)) (justify right))
+    )
+    (property "Value" "Varistor_6V" (id 1) (at 186.69 61.9767 0)
+      (effects (font (size 1.27 1.27)) (justify right))
+    )
+    (property "Footprint" "Capacitor_SMD:C_0805_2012Metric" (id 2) (at 188.722 60.96 90)
+      (effects (font (size 1.27 1.27)) hide)
+    )
+    (property "Datasheet" "~" (id 3) (at 190.5 60.96 0)
+      (effects (font (size 1.27 1.27)) hide)
+    )
+    (pin "1")
+    (pin "2")
+  )
+  (symbol (lib_id "power:+5V") (at 182.88 68.58 90) (mirror x) (unit 1)
+    (in_bom yes) (on_board yes)
+    (property "Reference" "#PWR03" (id 0) (at 186.69 68.58 0)
+      (effects (font (size 1.27 1.27)) hide)
+    )
+    (property "Value" "+5V" (id 1) (at 179.07 68.58 0))
+    (property "Footprint" "" (id 2) (at 182.88 68.58 0)
+      (effects (font (size 1.27 1.27)) hide)
+    )
+    (property "Datasheet" "" (id 3) (at 182.88 68.58 0)
       (effects (font (size 1.27 1.27)) hide)
     )
@@
     (pin "2")
   )
+  (symbol (lib_id "power:GND") (at 190.5 54.61 180) (unit 1)
+    (in_bom yes) (on_board yes)
+    (property "Reference" "#PWR0160" (id 0) (at 190.5 48.26 0)
+      (effects (font (size 1.27 1.27)) hide)
+    )
+    (property "Value" "GND" (id 1) (at 190.5 50.8 0))
+    (property "Footprint" "" (id 2) (at 190.5 54.61 0)
+      (effects (font (size 1.27 1.27)) hide)
+    )
+    (property "Datasheet" "" (id 3) (at 190.5 54.61 0)
+      (effects (font (size 1.27 1.27)) hide)
+    )
+    (pin "1")
+  )
   (symbol (lib_id "Switch:SW_DIP_x02") (at 80.01 71.12 0) (unit 1)
     (in_bom yes) (on_board yes) (fields_autoplaced)
@@
     )
     (property "Datasheet" "" (id 3) (at 146.05 115.57 0)
+      (effects (font (size 1.27 1.27)) hide)
+    )
+    (pin "1")
+  )
+  (symbol (lib_id "power:+5V") (at 233.68 68.58 270) (mirror x) (unit 1)
+    (in_bom yes) (on_board yes)
+    (property "Reference" "#PWR0159" (id 0) (at 229.87 68.58 0)
+      (effects (font (size 1.27 1.27)) hide)
+    )
+    (property "Value" "+5V" (id 1) (at 237.49 68.58 0))
+    (property "Footprint" "" (id 2) (at 233.68 68.58 0)
+      (effects (font (size 1.27 1.27)) hide)
+    )
+    (property "Datasheet" "" (id 3) (at 233.68 68.58 0)
       (effects (font (size 1.27 1.27)) hide)
     )
@@
       (reference "#PWR0158") (unit 1) (value "+5V") (footprint "")
     )
+    (path "/dc331e90-441a-4d41-b74d-22ef007a80d1"
+      (reference "#PWR0159") (unit 1) (value "+5V") (footprint "")
+    )
+    (path "/b0352ece-0814-496c-8434-0f30409d3ac7"
+      (reference "#PWR0160") (unit 1) (value "GND") (footprint "")
+    )
     (path "/b29395cc-df8a-4f64-b34d-9bd29e97e257/a7903183-69ad-4c1a-8f27-a148d44bc944"
       (reference "C1") (unit 1) (value "100nF") (footprint "Capacitor_SMD:C_0603_1608Metric")
@@
       (reference "L1") (unit 1) (value "4.7uH") (footprint "Inductor_SMD:L_Bourns_SRN6045TA")
     )
+    (path "/3f9a6295-6e64-4ee9-bb0b-9ab07bc61f16"
+      (reference "L2") (unit 1) (value "27n") (footprint "Inductor_SMD:L_0805_2012Metric")
+    )
     (path "/ba7b27e8-0e7e-4813-a1f3-426618b08ae4/e2cef837-fd7c-45f8-8139-0b4411c5636a"
       (reference "Q1") (unit 1) (value "IRF3205") (footprint "Package_TO_SOT_THT:TO-220-3_Vertical")
@@
       (reference "RV2") (unit 1) (value "10k") (footprint "Potentiometer_THT:Potentiometer_Bourns_3266Y_Vertical")
     )
+    (path "/6ec5c890-be35-4b4b-9f06-a0cb513b670d"
+      (reference "RV3") (unit 1) (value "Varistor_6V") (footprint "Capacitor_SMD:C_0805_2012Metric")
+    )
     (path "/b4604dc1-f8a2-492e-967c-482d1df18d8d"
