File: Proyecto Final (PCB)/Regulador 5V 2A.kicad_sch (KiCad schematic)
At the start: 6 parts, among them U7 AP63205WU

Commit message: Corrección en el aula
Connections:
- net SW: now reaches C10.1, L1.1, U7.5 (SW)
Changed lines of the file:
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@@
 (kicad_sch (version 20211123) (generator eeschema)
   (paper "A4")
+  (junction (at 147.32 102.87) (diameter 0) (color 0 0 0 0)
+  )
   (junction (at 113.03 107.95) (diameter 0) (color 0 0 0 0)
   )
@@
   )
   (junction (at 165.1 118.11) (diameter 0) (color 0 0 0 0)
-  )
-  (junction (at 147.32 102.87) (diameter 0) (color 0 0 0 0)
   )
   (junction (at 128.27 118.11) (diameter 0) (color 0 0 0 0)
@@
     (stroke (width 0) (type default) (color 0 0 0 0))
   )
-  (wire (pts (xy 138.43 102.87) (xy 147.32 102.87))
-    (stroke (width 0) (type default) (color 0 0 0 0))
-  )
   (wire (pts (xy 113.03 107.95) (xy 113.03 109.22))
-    (stroke (width 0) (type default) (color 0 0 0 0))
-  )
-  (wire (pts (xy 147.32 105.41) (xy 147.32 102.87))
     (stroke (width 0) (type default) (color 0 0 0 0))
   )
@@
     (stroke (width 0) (type default) (color 0 0 0 0))
   )
-  (wire (pts (xy 165.1 107.95) (xy 165.1 102.87))
+  (wire (pts (xy 147.32 102.87) (xy 148.59 102.87))
     (stroke (width 0) (type default) (color 0 0 0 0))
   )
-  (wire (pts (xy 147.32 102.87) (xy 148.59 102.87))
+  (wire (pts (xy 165.1 107.95) (xy 165.1 102.87))
     (stroke (width 0) (type default) (color 0 0 0 0))
   )
@@
   )
   (wire (pts (xy 128.27 113.03) (xy 128.27 118.11))
+    (stroke (width 0) (type default) (color 0 0 0 0))
+  )
+  (wire (pts (xy 138.43 102.87) (xy 147.32 102.87))
     (stroke (width 0) (type default) (color 0 0 0 0))
   )
@@
     (stroke (width 0) (type default) (color 0 0 0 0))
   )
+  (wire (pts (xy 147.32 105.41) (xy 147.32 102.87))
+    (stroke (width 0) (type default) (color 0 0 0 0))
+  )
   (wire (pts (xy 165.1 115.57) (xy 165.1 118.11))
     (stroke (width 0) (type default) (color 0 0 0 0))
@@
     (stroke (width 0) (type default) (color 0 0 0 0))
   )
+  (label "SW" (at 138.43 102.87 0)
+    (effects (font (size 1.27 1.27)) (justify left bottom))
+  )
   (symbol (lib_id "power:GND") (at 128.27 119.38 0) (unit 1)
