File: Proyecto Final (PCB)/Proyecto Final.kicad_pcb (KiCad board)
At the start: 2 copper layers, 133.5 x 71.2 mm, 55 parts, among them IC1 MC9S08MP16xLC, J1 Input, J10 Relay3, J11 Motor2, J12 Motor4, J13 LCD PINs, J14 Relay2, J15 Relay4, J16 PH_SENSOR, J17 Nivel_L, J18 Nivel_H, J19 Expansion2, J2 Luces_LEDs1, J20 Luces_LEDs2, J3 Expansions5, J4 DHT11_SENSOR, J5 LDR, J6 TDS_SENSOR, J7 Motor1, J8 Motor3, J9 Relay1, K1 FINDER-36.11, K2 FINDER-36.11, K3 FINDER-36.11, K4 FINDER-36.11, Q1 IRF3205, Q2 IRF3205, U1 AP63205WU, U2 MIC4427, U3 TLV2371D, U4 TLV2371D, U5 TLV2371D, U6 PC817, U7 PC817, U8 ULN2803A

Commit message: 02/07/2022
Parts:
- removed U5: TLV2371D, Package_SO:SOIC-8_3.9x4.9mm_P1.27mm
- added C10: 100nF, Capacitor_SMD:C_0603_1608Metric, F.Cu at (187.3, 91.2)
- added C11: 100nF, Capacitor_SMD:C_0603_1608Metric, F.Cu at (181.1, 80.8)
- added C12: 100nF, Capacitor_SMD:C_0603_1608Metric, F.Cu at (177.9, 80.8)
- added C9: 100nF, Capacitor_SMD:C_0603_1608Metric, F.Cu at (169.9, 91.9)
- added J21: Conn_01x04_Male, Connector_PinHeader_1.00mm:PinHeader_1x04_P1.00mm_Vertical, F.Cu at (178.2, 64.6)
- added R10: 5k, Resistor_SMD:R_0603_1608Metric, F.Cu at (156.6, 118.4)
- added R11: 10k, Resistor_SMD:R_0603_1608Metric, F.Cu at (150.4, 90.9)
- added R12: 10k, Resistor_SMD:R_0603_1608Metric, F.Cu at (150.2, 84.2)
- added R13: 10, Resistor_SMD:R_0603_1608Metric, F.Cu at (153.3, 90.9)
- added R14: 10, Resistor_SMD:R_0603_1608Metric, F.Cu at (153.2, 84.2)
- added R15: 1k, Resistor_SMD:R_0603_1608Metric, F.Cu at (208.2, 105.9)
- added R16: 5k, Resistor_SMD:R_0603_1608Metric, F.Cu at (148.3, 113.2)
- added R17: 5k, Resistor_SMD:R_0603_1608Metric, F.Cu at (156.7, 113.4)
- added R18: 5k, Resistor_SMD:R_0603_1608Metric, F.Cu at (153.8, 106.4)
- added R19: 5k, Resistor_SMD:R_0603_1608Metric, F.Cu at (153.8, 103.5)
- added R9: 5k, Resistor_SMD:R_0603_1608Metric, F.Cu at (148.0, 118.4)
- added RV2: 10k, Potentiometer_THT:Potentiometer_Bourns_3266Y_Vertical, F.Cu at (234.6, 118.5)
- added SW1: SWDIP, Button_Switch_THT:SW_DIP_SPSTx02_Slide_9.78x7.26mm_W7.62mm_P2.54mm, F.Cu at (140.1, 123.8)
- added U10: ULN2803A, Package_SO:SOIC-18W_7.5x11.6mm_P1.27mm, F.Cu at (175.1, 110.0)
- added Y1: Crystal, Crystal:Crystal_HC49-4H_Vertical, F.Cu at (163.4, 78.4)
- R1, R2: value 1k -> 10
- RV1: footprint Potentiometer_THT:Potentiometer_Bourns_3266W_Vertical -> Potentiometer_THT:Potentiometer_Bourns_3266Y_Vertical
- U3, U4: value TLV2371D -> LM358
- moved RV1 107.5 mm to (234.6, 110.4), turned to 90 degrees
- moved J1 88.2 mm to (125.6, 128.8)
- moved J7 75.7 mm to (182.5, 128.5), turned to 0 degrees
- moved J16 71.3 mm to (168.9, 67.8), turned to 180 degrees
- moved Q1 69.2 mm to (235.5, 129.1), turned to 180 degrees
- moved J18 69.0 mm to (214.6, 67.4), turned to 180 degrees
- moved J6 63.6 mm to (137.2, 67.8), turned to 180 degrees
- moved J11 63.0 mm to (170.8, 128.5), turned to 0 degrees
- moved J12 60.9 mm to (147.6, 128.5), turned to 0 degrees
- moved J17 60.4 mm to (203.8, 67.4), turned to 180 degrees
- moved J5 59.5 mm to (193.0, 67.4), turned to 180 degrees
- moved Q2 59.4 mm to (222.5, 129.1), turned to 180 degrees
- moved J4 59.1 mm to (153.0, 67.8), turned to 180 degrees
- moved J2 59.1 mm to (193.7, 128.5), turned to 0 degrees
- moved J20 58.9 mm to (204.7, 128.5), turned to 0 degrees
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Connections:
- net PTC0 renamed PWM_L2
- net PTC1 renamed PWM_L1
- IC1 pad 12: unconnected-(IC1-Pad12) -> Net-(IC1-Pad12)
- IC1 pad 13: SDA_e -> DIP1
- IC1 pad 14: SCL_e -> DIP2
- IC1 pad 15: Motor2 -> Motor3
- IC1 pad 16: Motor3 -> Motor2
- IC1 pad 21: unconnected-(IC1-Pad21) -> +5V
- IC1 pad 22: unconnected-(IC1-Pad22) -> GND
- IC1 pad 23: Motor4 -> Motor1
- IC1 pad 27: unconnected-(IC1-Pad27) -> Net-(IC1-Pad27)
- IC1 pad 28: unconnected-(IC1-Pad28) -> Net-(IC1-Pad28)
- IC1 pad 30: unconnected-(IC1-Pad30) -> Net-(IC1-Pad30)
- IC1 pad 5: Motor1 -> Motor4
- J2 pad 1: +12V -> Net-(Q1-Pad2)
- J2 pad 2: Net-(Q1-Pad2) -> +12V
- J3 pad 3: SDA_e -> SCL
- J3 pad 4: SCL_e -> SDA
- J3 pad 5: ADC_e -> Net-(J3-Pad5)
- RV1 pad 1: GND -> Net-(U6-Pad1)
- RV1 pad 2: GND -> Net-(U6-Pad1)
- RV1 pad 3: Net-(J5-Pad2) -> Net-(J17-Pad2)
- U2 pad 6: +5V -> +12V
- U3 pad 1: unconnected-(U3-Pad1) -> Net-(R4-Pad2)
- U3 pad 5: unconnected-(U3-Pad5) -> Net-(J3-Pad5)
- U3 pad 6: Net-(R4-Pad2) -> Net-(R15-Pad2)
- U3 pad 7: +5V -> Net-(R15-Pad2)
- U3 pad 8: unconnected-(U3-Pad8) -> +5V
- U4 pad 1: unconnected-(U4-Pad1) -> Net-(R6-Pad2)
- U4 pad 2: Net-(R5-Pad2) -> Net-(R6-Pad2)
- U4 pad 3: Net-(J6-Pad3) -> Net-(J16-Pad3)
- U4 pad 5: unconnected-(U4-Pad5) -> Net-(J6-Pad3)
- U4 pad 7: +5V -> Net-(R5-Pad2)
- U4 pad 8: unconnected-(U4-Pad8) -> +5V
- U6 pad 1: Net-(R9-Pad1) -> Net-(U6-Pad1)
- U7 pad 1: Net-(R10-Pad1) -> Net-(U7-Pad1)
- U8 pad 1: Motor4 -> Relay4
- U8 pad 11: M4 -> unconnected-(U8-Pad11)
- U8 pad 12: M3 -> unconnected-(U8-Pad12)
- U8 pad 13: M2 -> unconnected-(U8-Pad13)
- U8 pad 14: M1 -> unconnected-(U8-Pad14)
- U8 pad 2: Motor3 -> Relay3
- U8 pad 3: Motor2 -> Relay2
- U8 pad 4: Motor1 -> Relay1
- U8 pad 5: Relay4 -> unconnected-(U8-Pad5)
- U8 pad 6: Relay3 -> unconnected-(U8-Pad6)
- U8 pad 7: Relay2 -> unconnected-(U8-Pad7)
- U8 pad 8: Relay1 -> unconnected-(U8-Pad8)
Other:
- board size 133.5 x 71.2 mm -> 150 x 72 mm

Commit message: 02/07/2022
Parts:
- removed the R10 at (202.9, 97.5)
- removed the R9 at (207.6, 97.7)
Routing:
- net +5V: track 0.00 -> 339.6 mm
- net +12V: track 0.00 -> 240.8 mm
- net SDA: track 0.00 -> 160.4 mm
- net Net-(Q1-Pad1): track 0.00 -> 148.5 mm
- net SCL: track 0.00 -> 137.6 mm
- net Net-(J6-Pad3): track 0.00 -> 96.0 mm, vias 0 -> 1
- net Net-(Q2-Pad1): track 0.00 -> 90.7 mm, vias 0 -> 1
- net Rx: track 0.00 -> 90.2 mm, vias 0 -> 2
- net Tx: track 0.00 -> 86.8 mm, vias 0 -> 2
- net DIP1: track 0.00 -> 68.3 mm, vias 0 -> 1
- net DIP2: track 0.00 -> 67.7 mm, vias 0 -> 1
- net Net-(J18-Pad2): track 0.00 -> 67.4 mm
- net Net-(J3-Pad5): track 0.00 -> 65.8 mm
- net Net-(J16-Pad3): track 0.00 -> 63.6 mm, vias 0 -> 1
- net Net-(J17-Pad2): track 0.00 -> 62.9 mm
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
Commit message: 08/07/2022
Parts:
- J13, J21: footprint Connector_PinHeader_1.00mm:PinHeader_1x04_P1.00mm_Vertical -> Connector_PinHeader_2.54mm:PinHeader_1x04_P2.54mm_Vertical
- moved J13 9.61 mm to (226.7, 102.2)
- moved J21 4.14 mm to (182.2, 65.3)

Commit message: 14/07/2022
Parts:
- removed U8: ULN2803A, Package_SO:SOIC-18W_7.5x11.6mm_P1.27mm
- added C13: 30pF, Capacitor_SMD:C_0603_1608Metric, F.Cu at (196.1, 105.5)
- added C14: 30pF, Capacitor_SMD:C_0603_1608Metric, F.Cu at (196.1, 103.6)
- added C15: 100n, Capacitor_SMD:C_0201_0603Metric, F.Cu at (150.7, 115.8)
- added C16: 100n, Capacitor_SMD:C_0201_0603Metric, F.Cu at (107.7, 122.7)
- added C17: 4.7µ, Capacitor_SMD:C_0805_2012Metric, F.Cu at (229.4, 91.2)
- added C18: 100n, Capacitor_SMD:C_0201_0603Metric, F.Cu at (232.6, 91.2)
- added R20: 1M, Resistor_SMD:R_0201_0603Metric, F.Cu at (203.5, 104.4)
- added U5: MIC4427, Package_SO:SOIC-8_3.9x4.9mm_P1.27mm, F.Cu at (225.0, 91.2)
- C1: value 10uF -> 100nF
- C10: footprint Capacitor_SMD:C_0603_1608Metric -> Capacitor_SMD:C_0201_0603Metric
- C11: value 100nF -> 22uF; footprint Capacitor_SMD:C_0603_1608Metric -> Capacitor_SMD:C_0805_2012Metric
- C12: value 100nF -> 22uf; footprint Capacitor_SMD:C_0603_1608Metric -> Capacitor_SMD:C_0805_2012Metric
- C3: value 22uF -> 100nF
- C4: value 22uf -> 100nF
- C8: value 100nF -> 10uF; footprint Capacitor_SMD:C_0603_1608Metric -> Capacitor_SMD:C_0805_2012Metric
- J10: value Relay3 -> Expansions5; footprint TerminalBlock:TerminalBlock_bornier-3_P5.08mm -> TerminalBlock:TerminalBlock_bornier-5_P5.08mm
- J13: value LCD PINs -> Expansion2; footprint Connector_PinHeader_2.54mm:PinHeader_1x04_P2.54mm_Vertical -> TerminalBlock:TerminalBlock_bornier-2_P5.08mm
- J14: value Relay2 -> Luces_LEDs1; footprint TerminalBlock:TerminalBlock_bornier-3_P5.08mm -> TerminalBlock:TerminalBlock_bornier-2_P5.08mm
- J15: value Relay4 -> Luces_LEDs2; footprint TerminalBlock:TerminalBlock_bornier-3_P5.08mm -> TerminalBlock:TerminalBlock_bornier-2_P5.08mm
- J16: value PH_SENSOR -> Relay1
- J17: value Nivel_L -> Relay3; footprint TerminalBlock:TerminalBlock_bornier-2_P5.08mm -> TerminalBlock:TerminalBlock_bornier-3_P5.08mm
- J18: value Nivel_H -> Relay2; footprint TerminalBlock:TerminalBlock_bornier-2_P5.08mm -> TerminalBlock:TerminalBlock_bornier-3_P5.08mm
- J19: value Expansion2 -> Relay4; footprint TerminalBlock:TerminalBlock_bornier-2_P5.08mm -> TerminalBlock:TerminalBlock_bornier-3_P5.08mm
- J2: value Luces_LEDs1 -> DHT11_SENSOR; footprint TerminalBlock:TerminalBlock_bornier-2_P5.08mm -> TerminalBlock:TerminalBlock_bornier-3_P5.08mm
- J20: value Luces_LEDs2 -> LCD PINs; footprint TerminalBlock:TerminalBlock_bornier-2_P5.08mm -> Connector_PinHeader_2.54mm:PinHeader_1x04_P2.54mm_Vertical
- J3: value Expansions5 -> LDR; footprint TerminalBlock:TerminalBlock_bornier-5_P5.08mm -> TerminalBlock:TerminalBlock_bornier-2_P5.08mm
- J4: value DHT11_SENSOR -> TDS_SENSOR
- J5: value LDR -> PH_SENSOR; footprint TerminalBlock:TerminalBlock_bornier-2_P5.08mm -> TerminalBlock:TerminalBlock_bornier-3_P5.08mm
- J6: value TDS_SENSOR -> Nivel_L; footprint TerminalBlock:TerminalBlock_bornier-3_P5.08mm -> TerminalBlock:TerminalBlock_bornier-2_P5.08mm
- J9: value Relay1 -> Nivel_H; footprint TerminalBlock:TerminalBlock_bornier-3_P5.08mm -> TerminalBlock:TerminalBlock_bornier-2_P5.08mm
- L1: footprint Inductor_SMD:L_0603_1608Metric -> Inductor_SMD:L_Bourns_SRN6045TA
- R1, R13: value 10 -> 5k
- R11, R12: value 10k -> 5k
- R14: value 10 -> 10k
- R15: value 1k -> 10k
- R16, R17, R18, R19: value 5k -> 10
- R2: value 10 -> 1k
- R3, R7: value 5k -> 1k
- R5, R6: value 1k -> 5k
- U1: value AP63205WU -> LM358; footprint Package_TO_SOT_SMD:TSOT-23-6 -> Package_SO:SOIC-8_3.9x4.9mm_P1.27mm
- U10: value ULN2803A -> ULN2003A; footprint Package_SO:SOIC-18W_7.5x11.6mm_P1.27mm -> Package_SO:SOIC-16_3.9x9.9mm_P1.27mm
- U2: value MIC4427 -> LM358
- U3, U4: value LM358 -> PC817; footprint Package_SO:SOIC-8_3.9x4.9mm_P1.27mm -> Package_DIP:DIP-4_W7.62mm
- U6: value PC817 -> ULN2003A; footprint Package_DIP:DIP-4_W7.62mm -> Package_SO:SOIC-16_3.9x9.9mm_P1.27mm
- U7: value PC817 -> AP63205WU; footprint Package_DIP:DIP-4_W7.62mm -> Package_TO_SOT_SMD:TSOT-23-6
- moved J14 132.5 mm to (225.6, 69.3), turned to 180 degrees
- moved J15 118.0 mm to (215.1, 69.3), turned to 180 degrees
- moved J10 117.0 mm to (205.6, 129.0), turned to 0 degrees
- moved J1 106.0 mm to (231.6, 129.0)
- moved L1 104.0 mm to (230.5, 115.6), turned to 0 degrees
- moved J5 101.7 mm to (112.1, 129.0), turned to 0 degrees
- moved J3 99.7 mm to (143.6, 129.0), turned to 0 degrees
- moved R3 93.8 mm to (103.0, 117.6), turned to -90 degrees
- moved J18 92.5 mm to (122.2, 69.3)
- moved R16 87.9 mm to (230.6, 82.3), turned to 0 degrees
- moved J19 84.2 mm to (155.2, 69.3), turned to 180 degrees
- moved J4 83.3 mm to (96.5, 129.0), turned to 0 degrees
- moved U6 81.4 mm to (130.9, 98.8), turned to 90 degrees
- moved J12 81.0 mm to (202.8, 69.3), turned to 180 degrees
- moved RV2 79.3 mm to (157.2, 101.5), turned to -90 degrees
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Connections:
- C1 pad 1: +12V -> LDR_SENSOR
- C10 pad 1: ADC_e -> Net-(C10-Pad1)
- C10 pad 2: GND -> Net-(C10-Pad2)
- C11 pad 1: GND -> +5V
- C11 pad 2: LEVEL_L -> GND
- C12 pad 1: GND -> +5V
- C12 pad 2: LEVEL_H -> GND
- C2 pad 1: Net-(C2-Pad1) -> OUT_TDS
- C2 pad 2: Net-(C2-Pad2) -> GND
- C3 pad 1: +5V -> OUT_PH
- C4 pad 1: +5V -> GND
- C4 pad 2: GND -> LEVEL_L
- C5 pad 1: LDR_SENSOR -> GND
- C5 pad 2: GND -> LEVEL_H
- C7 pad 1: OUT_TDS -> ADC_e
- C8 pad 1: OUT_PH -> +12V
- J10 pad 1: NO_Relay3 -> Tx
- J10 pad 2: C_Relay3 -> Rx
- J10 pad 3: NC_Relay3 -> SCL
- J13 pad 1: GND -> +5V
- J13 pad 2: +5V -> GND
- J14 pad 1: NO_Relay2 -> Net-(J14-Pad1)
- J14 pad 2: C_Relay2 -> +12V
- J15 pad 1: NO_Relay4 -> +12V
- J15 pad 2: C_Relay4 -> Net-(J15-Pad2)
- J16 pad 1: GND -> NO_Relay1
- J16 pad 2: +5V -> C_Relay1
- J16 pad 3: Net-(J16-Pad3) -> NC_Relay1
- J17 pad 1: +5V -> NO_Relay3
- J17 pad 2: Net-(J17-Pad2) -> C_Relay3
- J18 pad 1: +5V -> NO_Relay2
- J18 pad 2: Net-(J18-Pad2) -> C_Relay2
- J19 pad 1: +5V -> NO_Relay4
- J19 pad 2: GND -> C_Relay4
- J2 pad 1: Net-(Q1-Pad2) -> GND
- J2 pad 2: +12V -> +5V
- J20 pad 1: +12V -> GND
- J20 pad 2: Net-(Q2-Pad2) -> +5V
- J3 pad 1: Tx -> +5V
- J3 pad 2: Rx -> Net-(J3-Pad2)
- J4 pad 3: OUT_DHT11 -> Net-(J4-Pad3)
- J5 pad 1: +5V -> GND
- J5 pad 2: Net-(J5-Pad2) -> +5V
- J6 pad 1: GND -> +5V
- J6 pad 2: +5V -> Net-(J6-Pad2)
- J9 pad 1: NO_Relay1 -> +5V
- J9 pad 2: C_Relay1 -> Net-(J9-Pad2)
- L1 pad 1: Net-(C2-Pad1) -> Net-(C10-Pad1)
- Q1 pad 2: Net-(Q1-Pad2) -> Net-(J14-Pad1)
- Q2 pad 2: Net-(Q2-Pad2) -> Net-(J15-Pad2)
- R1 pad 1: Net-(Q1-Pad1) -> OUT_DHT11
- R1 pad 2: Net-(R1-Pad2) -> +5V
- R11 pad 1: Net-(Q1-Pad1) -> +5V
- R11 pad 2: GND -> SCL
- R12 pad 1: GND -> +5V
- R12 pad 2: Net-(Q2-Pad1) -> Rx
- R13 pad 1: Net-(Q1-Pad1) -> +5V
- R13 pad 2: Net-(R1-Pad2) -> Tx
- R14 pad 1: Net-(Q2-Pad1) -> Net-(Q1-Pad1)
- R14 pad 2: Net-(R14-Pad2) -> GND
- R15 pad 1: ADC_e -> GND
- R15 pad 2: Net-(R15-Pad2) -> Net-(Q2-Pad1)
- R16 pad 1: +5V -> Net-(Q1-Pad1)
- R16 pad 2: SDA -> Net-(R16-Pad2)
- R17 pad 1: +5V -> Net-(Q1-Pad1)
- R17 pad 2: SCL -> Net-(R16-Pad2)
- R18 pad 1: +5V -> Net-(Q2-Pad1)
- R18 pad 2: Rx -> Net-(R18-Pad2)
- R19 pad 1: +5V -> Net-(Q2-Pad1)
- R19 pad 2: Tx -> Net-(R18-Pad2)
- R2 pad 1: Net-(Q2-Pad1) -> LDR_SENSOR
- R2 pad 2: Net-(R14-Pad2) -> Net-(R2-Pad2)
- R3 pad 1: OUT_DHT11 -> OUT_TDS
- R3 pad 2: +5V -> Net-(R3-Pad2)
- R4 pad 1: LDR_SENSOR -> OUT_PH
- R5 pad 1: OUT_TDS -> +5V
- R5 pad 2: Net-(R5-Pad2) -> LEVEL_L
- R6 pad 1: OUT_PH -> +5V
- R6 pad 2: Net-(R6-Pad2) -> LEVEL_H
- R7 pad 1: +5V -> ADC_e
- R7 pad 2: LEVEL_L -> Net-(R7-Pad2)
- R8 pad 2: LEVEL_H -> SDA
- RV1 pad 1: Net-(U6-Pad1) -> Net-(RV1-Pad1)
- RV1 pad 2: Net-(U6-Pad1) -> Net-(RV1-Pad1)
- RV1 pad 3: Net-(J17-Pad2) -> Net-(J6-Pad2)
- RV2 pad 1: Net-(U7-Pad1) -> Net-(RV2-Pad1)
- RV2 pad 2: Net-(U7-Pad1) -> Net-(RV2-Pad1)
- RV2 pad 3: Net-(J18-Pad2) -> Net-(J9-Pad2)
- U1 pad 1: +5V -> Net-(R4-Pad2)
- U1 pad 2: +12V -> Net-(R4-Pad2)
- U1 pad 3: +12V -> Net-(J5-Pad3)
- U1 pad 5: Net-(C2-Pad1) -> Net-(J4-Pad3)
- U1 pad 6: Net-(C2-Pad2) -> Net-(R3-Pad2)
- U10 pad 10: +12V -> M4
- U10 pad 11: M4 -> M3
- U10 pad 12: M4 -> M3
- U10 pad 13: M3 -> M2
- U10 pad 14: M3 -> M2
- U10 pad 15: M2 -> M1
- U10 pad 16: M2 -> M1
- U10 pad 8: Motor4 -> GND
- U10 pad 9: GND -> +12V
- U2 pad 1: unconnected-(U2-Pad1) -> Net-(R2-Pad2)
- U2 pad 2: PWM_L1 -> Net-(R2-Pad2)
- U2 pad 3: GND -> Net-(J3-Pad2)
- U2 pad 4: PWM_L2 -> GND
- U2 pad 5: Net-(R14-Pad2) -> Net-(J10-Pad5)
- U2 pad 6: +12V -> Net-(R7-Pad2)
- U2 pad 7: Net-(R1-Pad2) -> Net-(R7-Pad2)
- U2 pad 8: unconnected-(U2-Pad8) -> +5V
- U3 pad 1: Net-(R4-Pad2) -> Net-(RV1-Pad1)
- U3 pad 2: Net-(R4-Pad2) -> GND
- U3 pad 3: Net-(J5-Pad2) -> GND
- U3 pad 4: GND -> LEVEL_L
- U4 pad 1: Net-(R6-Pad2) -> Net-(RV2-Pad1)
- U4 pad 2: Net-(R6-Pad2) -> GND
- U4 pad 3: Net-(J16-Pad3) -> GND
- U4 pad 4: GND -> LEVEL_H
- U6 pad 1: Net-(U6-Pad1) -> Relay4
- U6 pad 2: GND -> Relay3
- U6 pad 3: GND -> Relay2
- U6 pad 4: LEVEL_L -> Relay1
- U7 pad 1: Net-(U7-Pad1) -> +5V
- U7 pad 2: GND -> +12V
- U7 pad 3: GND -> +12V
- U7 pad 4: LEVEL_H -> GND
Routing:
- net +5V: track 339.6 -> 0.00 mm
- net +12V: track 240.8 -> 0.00 mm
- net SDA: track 160.4 -> 0.00 mm
- net Net-(Q1-Pad1): track 148.5 -> 0.00 mm
- net SCL: track 137.6 -> 0.00 mm
- net Net-(J6-Pad3): track 96.0 -> 0.00 mm, vias 1 -> 0
- net Net-(Q2-Pad1): track 90.7 -> 0.00 mm, vias 1 -> 0
- net Rx: track 90.2 -> 0.00 mm, vias 2 -> 0
- net Tx: track 86.8 -> 0.00 mm, vias 2 -> 0
- net DIP1: track 68.3 -> 0.00 mm, vias 1 -> 0
- net DIP2: track 67.7 -> 0.00 mm, vias 1 -> 0
- net Net-(J18-Pad2): track 67.4 -> 0.00 mm
- net Net-(J3-Pad5): track 65.8 -> 0.00 mm
- net Net-(J16-Pad3): track 63.6 -> 0.00 mm, vias 1 -> 0
- net Net-(J17-Pad2): track 62.9 -> 0.00 mm
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- added copper zone on In2.Cu, net +12V
- added copper zone on In2.Cu, net +5V
- added copper zone on In1.Cu, net GND
- removed copper zone on B.Cu, net GND
Other:
- copper layers 2 -> 4

Commit message: 15/07/2022
Parts:
- added L2: 27n, Inductor_SMD:L_0805_2012Metric, F.Cu at (189.1, 113.3)
- added RV3: Varistor_6V, Capacitor_SMD:C_0805_2012Metric, F.Cu at (182.2, 97.4)
- moved C1 3.33 mm to (184.0, 112.0)
- moved C2 3.33 mm to (182.1, 112.0)
- moved C3 3.33 mm to (180.2, 112.0)
- moved C7 3.33 mm to (185.9, 112.0)
- moved U6 1.95 mm to (131.1, 100.8)
- turned R10 to -90 degrees
Connections:
- C10 pad 1: Net-(C10-Pad1) -> GND
- C9 pad 2: +5V -> Net-(C9-Pad2)
- IC1 pad 21: +5V -> Net-(C9-Pad2)
- L1 pad 1: Net-(C10-Pad1) -> GND
- U7 pad 5: Net-(C10-Pad1) -> GND
Routing:
- net GND: track 0.00 -> 183.1 mm, vias 0 -> 13
- net +5V: track 0.00 -> 124.3 mm, vias 0 -> 9
- net +12V: track 0.00 -> 109.3 mm, vias 0 -> 2
- net OUT_TDS: track 0.00 -> 90.5 mm, vias 0 -> 2
- net Net-(J10-Pad5): track 0.00 -> 84.6 mm, vias 0 -> 3
- net SDA: track 0.00 -> 78.8 mm, vias 0 -> 3
- net OUT_PH: track 0.00 -> 77.6 mm, vias 0 -> 4
- net Relay3: track 0.00 -> 73.4 mm, vias 0 -> 6
- net Relay4: track 0.00 -> 73.3 mm, vias 0 -> 8
- net OUT_DHT11: track 0.00 -> 71.4 mm, vias 0 -> 4
- net SCL: track 0.00 -> 69.7 mm, vias 0 -> 3
- net Relay1: track 0.00 -> 67.8 mm, vias 0 -> 2
- net Relay2: track 0.00 -> 65.4 mm, vias 0 -> 2
- net LDR_SENSOR: track 0.00 -> 54.3 mm, vias 0 -> 6
- net LEVEL_H: track 0.00 -> 54.2 mm, vias 0 -> 5
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
Commit message: Corrección en el aula
Parts:
- moved C13 14.1 mm to (210.2, 105.5)
- moved C14 14.1 mm to (210.2, 103.6)
- moved C12 13.8 mm to (219.5, 111.9), turned to 90 degrees
- moved C11 13.8 mm to (222.0, 111.9), turned to 90 degrees
- moved L1 6.41 mm to (226.4, 110.6), turned to -90 degrees
- moved Y1 5.21 mm to (203.2, 102.7)
- moved C10 4.40 mm to (232.2, 107.6), turned to 180 degrees
- moved C8 4.27 mm to (236.0, 110.2), turned to 90 degrees
- moved R20 4.25 mm to (207.7, 104.5)
- moved RV1 1.05 mm to (157.5, 113.7)
- moved RV2 0.27 mm to (157.2, 101.2)
- turned U7 to 90 degrees
Connections:
- C10 pad 1: GND -> /Fuente SW/SW
- L1 pad 1: GND -> /Fuente SW/SW
- U7 pad 5: GND -> /Fuente SW/SW
Routing:
- net GND: track 183.1 -> 264.9 mm, vias 13 -> 24
- net +12V: track 109.3 -> 120.8 mm, vias 2 -> 3
- net +5V: track 124.3 -> 131.6 mm, vias 9 -> 28
- net Net-(C13-Pad2): track 18.7 -> 21.7 mm, vias 2 -> 0
- net /Fuente SW/SW: track 0.00 -> 2.25 mm
- net Relay4: track 73.3 -> 75.4 mm
- net Relay3: track 73.4 -> 75.2 mm
- net Net-(C10-Pad2): track 2.98 -> 1.51 mm
- net Relay2: track 65.4 -> 66.8 mm
- net Rele4: track 21.2 -> 19.9 mm, vias 1 -> 0
- net Net-(C14-Pad2): track 19.4 -> 20.7 mm, vias 4 -> 0
- net OUT_TDS: track 90.5 -> 89.8 mm
- net Rele1: track 39.5 -> 38.8 mm, vias 1 -> 0
- net Rele2: track 23.8 -> 23.2 mm, vias 1 -> 0
- net Rele3: vias 1 -> 0
- added copper zone on F.Cu, net +5V
- added copper zone on F.Cu, net /Fuente SW/SW
- added copper zone on F.Cu, net GND

Commit message: 22/07/2022
Routing:
- net +12V: track 120.8 -> 107.8 mm, vias 3 -> 1
- net +5V: track 131.6 -> 120.0 mm
- net Net-(IC1-Pad12): track 34.0 -> 28.8 mm, vias 4 -> 1
- net OUT_PH: track 77.6 -> 76.4 mm, vias 4 -> 2
- net LEVEL_L: track 47.9 -> 48.1 mm, vias 7 -> 4
- net PWM_L2: vias 2 -> 0
- net Net-(R16-Pad2): vias 2 -> 0
- net PWM_L1: vias 2 -> 0
- net LDR_SENSOR: vias 6 -> 4

Commit message: 22/07/2022 AULA
Routing:
- net +12V: track 107.8 -> 117.3 mm, vias 1 -> 0
- net LEVEL_H: track 54.2 -> 57.4 mm, vias 5 -> 4
- net Rx: track 50.9 -> 49.1 mm
- net Relay3: track 75.2 -> 76.0 mm, vias 6 -> 4
