File: Proyecto Final (PCB)/Proyecto Final.kicad_pcb (KiCad board)
At the start: 4 copper layers, 150 x 72 mm, 81 parts, among them IC1 MC9S08MP16xLC, J1 Input, J10 Expansions5, J11 Motor2, J12 Motor4, J13 Expansion2, J14 Luces_LEDs1, J15 Luces_LEDs2, J16 Relay1, J17 Relay3, J18 Relay2, J19 Relay4, J2 DHT11_SENSOR, J20 LCD PINs, J21 Conn_01x04_Male, J3 LDR, J4 TDS_SENSOR, J5 PH_SENSOR, J6 Nivel_L, J7 Motor1, J8 Motor3, J9 Nivel_H, K1 FINDER-36.11, K2 FINDER-36.11, K3 FINDER-36.11, K4 FINDER-36.11, Q1 IRF3205, Q2 IRF3205, SW1 SWDIP, U1 LM358, U10 ULN2003A, U2 LM358, U3 PC817, U4 PC817, U5 MIC4427, U6 ULN2003A, U7 AP63205WU, Y1 Crystal

Commit message: 5.02
Routing:
- net Net-(IC1-Pad30): track 42.0 -> 43.9 mm
- net DIP1: track 33.9 -> 34.9 mm
- net ADC_e: track 43.7 -> 43.0 mm
- net Net-(J6-Pad2): track 32.3 -> 32.8 mm

Commit message: 5.57
Other:
- board text added: "+12V"
- board text added: "+5V"
- board text added: "Comun"
- board text added: "DTH11"
- board text added: "GND"
- board text added: "HIGH L"
- board text added: "LDR"
- board text added: "LOW L"
- board text added: "NC"
- board text added: "NO"
- board text added: "Ph"
- board text added: "Rx"
- board text added: "SCL"
- board text added: "SDA"
- board text added: "TDS"
- board text added: "Tx"

Commit message: 6.28
Other:
- board text added: "-LEDs1"
- board text added: "-LEDs2"
- board text added: "-Motor1"
- board text added: "-Motor2"
- board text added: "-Motor3"
- board text added: "-Motor4"
- board text added: "1A"
- board text added: "500mA"
- board text added: "ADC"
- board text added: "BKGD"
- board text added: "LCD"
- board text added: "PRGM"
- board text added: "~RESET"

Commit message: 6.36
Other:
- board text added: "HIGH-LVL"
- board text added: "LOW-LVL"
- board text removed: "HIGH L"
- board text removed: "LOW L"
Changed lines of the file:
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@@
     (effects (font (size 0.762 0.762) (thickness 0.127)))
   )
-  (gr_text "HIGH L" (at 159.385 133.858) (layer "F.SilkS")
-    (effects (font (size 0.762 0.762) (thickness 0.127)))
+  (gr_text "HIGH-LVL" (at 159.385 133.858) (layer "F.SilkS")
+    (effects (font (size 0.635 0.635) (thickness 0.1016)))
   )
   (gr_text "-Motor3" (at 186.055 64.77) (layer "F.SilkS")
@@
     (effects (font (size 0.762 0.762) (thickness 0.127)))
   )
-  (gr_text "LOW L" (at 170.18 133.858) (layer "F.SilkS")
-    (effects (font (size 0.762 0.762) (thickness 0.127)))
+  (gr_text "LOW-LVL" (at 170.18 133.858) (layer "F.SilkS")
+    (effects (font (size 0.635 0.635) (thickness 0.1016)))
   )
   (gr_text "SCL" (at 215.9 133.8326) (layer "F.SilkS")
@@
     (pts (xy 91.186 62.493) (xy 241.186 62.493))
     (height -12.455)
-    (gr_text "5905.5118 mils" (at 166.186 48.238) (layer "F.Cu")
+    (gr_text "150.0000 mm" (at 166.186 48.238) (layer "F.Cu")
       (effects (font (size 1.5 1.5) (thickness 0.3)))
     )
-    (format (units 3) (units_format 1) (precision 4))
+    (format (units 2) (units_format 1) (precision 4))
     (style (thickness 0.2) (arrow_length 1.27) (text_position_mode 0) (extension_height 0.58642) (extension_offset 0.5) keep_text_aligned)
   )
@@
     (pts (xy 91.186 134.493) (xy 91.186 62.493))
     (height -9.779)
-    (gr_text "2834.6457 mils" (at 79.607 98.493 90) (layer "F.Cu")
+    (gr_text "72.0000 mm" (at 79.607 98.493 90) (layer "F.Cu")
       (effects (font (size 1.5 1.5) (thickness 0.3)))
     )
-    (format (units 3) (units_format 1) (precision 4))
+    (format (units 2) (units_format 1) (precision 4))
     (style (thickness 0.2) (arrow_length 1.27) (text_position_mode 0) (extension_height 0.58642) (extension_offset 0.5) keep_text_aligned)
   )

Commit message: 18:12
Parts:
- J10 (Expansiones): renamed from J10
Changed lines of the file:
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@@
     (property "Sheetname" "Expansions")
     (attr through_hole)
-    (fp_text reference "J13" (at 2.54 -4.699) (layer "F.SilkS")
-      (effects (font (size 1 1) (thickness 0.15)))
+    (fp_text reference "J13" (at 2.351 -4.432) (layer "F.SilkS")
+      (effects (font (size 0.635 0.635) (thickness 0.0762)))
     )
     (fp_text value "Expansion2" (at 2.54 5.08) (layer "F.Fab")
@@
     (property "Sheetname" "Expansions")
     (attr through_hole)
-    (fp_text reference "J10" (at 8.128 -4.699) (layer "F.SilkS")
-      (effects (font (size 1 1) (thickness 0.15)))
+    (fp_text reference "J10 (Expansiones)" (at 8.387 -4.482) (layer "F.SilkS")
+      (effects (font (size 0.635 0.635) (thickness 0.0762)))
     )
     (fp_text value "Expansions5" (at 10.15 4.6) (layer "F.Fab")
@@
     )
   )
-  (gr_rect (start 192.659 133.1214) (end 228.473 134.3406) (layer "F.SilkS") (width 0.0508) (fill none))
+  (gr_rect (start 192.209 124.0714) (end 228.823 134.3406) (layer "F.SilkS") (width 0.0508) (fill none))
   (gr_rect (start 91.186 134.493) (end 241.186 62.493) (layer "Edge.Cuts") (width 0.1) (fill none))
   (gr_text "500mA" (at 200.406 63.627) (layer "F.SilkS")

Commit message: 28-07-2022
Other:
- board text added: "Jorge Nicolas 2019-8447"
Changed lines of the file:
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@@
     (effects (font (size 0.762 0.762) (thickness 0.127)))
+  )
+  (gr_text "Jorge Nicolas \n2019-8447" (at 235.585 65.405) (layer "F.SilkS")
+    (effects (font (size 1 1) (thickness 0.15)))
   )
   (gr_text "+5V" (at 101.092 133.858) (layer "F.SilkS")

Commit message: 24/08/2022
Parts:
- added J3: Conn_01x20_Male, Connector_PinSocket_2.54mm:PinSocket_1x20_P2.54mm_Vertical, F.Cu at (151.1, 159.6)
- added J4: Conn_01x20_Male, Connector_PinSocket_2.54mm:PinSocket_1x20_P2.54mm_Vertical, F.Cu at (102.9, 144.4)

Commit message: 25/08/2022
Parts:
- removed the J3 at (151.1, 159.6)
- removed the J4 at (102.9, 144.4)
